File: 02.Hardware/PCBs/Carrier General/Carrier Motor Driver.sch (EAGLE design)
At the start: 87 parts, among them IC1 MCP6001T-I_LT, IC2 AP62200WU-7, IC3 PCF8575DB, U1 MCP6002T-I/SN, U2 LM4040BIM3-2.0/NOPB, U3 ATE1D-5M3-10-Z

Commit message: Se añade 3v3 para filtro ISENSE + Cambios menores
Parts:
- removed IC1: MCP6001T-I_LT, MCP6001T-I_LT:MCP6001T-I_LT
- removed U$1: (no value), RaspberryPi_Pico:RPI_PICO_IG-SMD
- added ENA: TESTPAD_TPSQPAD1-17, BeagleBone_Blue_R3:TESTPAD_TPSQPAD1-17
- added U4: (no value), RaspberryPi_Pico:RPI_PICO_IG-SMD
- added U5: MCP6001T-I_LT, MCP6001T-I_LT:MCP6001T-I_LT
Connections:
- net DSP_RST: now also U4.GP15; no longer U$1.GP15
- net EN_0: now also U4.GP9; no longer U$1.GP9
- net EN_1: now also U4.GP11; no longer U$1.GP11
- net EN_2: now also U4.GP3; no longer U$1.GP3
- net EN_3: now also U4.GP7; no longer U$1.GP7
- net EN_4: now also U4.GP21; no longer U$1.GP21
- net EN_5: now also U4.GP1; no longer U$1.GP1
- net EN_DCDC: now also ENA.TP
- net GND: now also IC3.A0, IC3.A1, IC3.A2, U4.GND@1, U4.GND@2, U4.GND@3, U4.GND@4, U4.GND@6, U4.GND@7, U4.GND@8, U5.VSS; no longer IC1.VSS, OUT_MOTOR_DRIVER.10, U$1.GND@1, U$1.GND@2, U$1.GND@3, U$1.GND@4, U$1.GND@6, U$1.GND@7, U$1.GND@8
- net ISENSE: now also U4.GP28_A2; no longer U$1.GP28_A2
- net MISO: now also U4.GP16; no longer U$1.GP16
- net MOSI: now also U4.GP19; no longer U$1.GP19
- net N$6: now also U5.VIN-; no longer IC1.VIN-
- net N$8: now also U5.VIN+; no longer IC1.VIN+
- net PWM_IN_0: now also U4.GP8; no longer U$1.GP8
- net PWM_IN_1: now also U4.GP10; no longer U$1.GP10
- net PWM_IN_2: now also U4.GP2; no longer U$1.GP2
- net PWM_IN_3: now also U4.GP6; no longer U$1.GP6
- net PWM_IN_4: now also U4.GP22; no longer U$1.GP22
- net PWM_IN_5: now also U4.GP20; no longer U$1.GP20
- net SCK: now also U4.GP18; no longer U$1.GP18
- net SCL: now also U4.GP5; no longer U$1.GP5
- net SDA: now also U4.GP4; no longer U$1.GP4
- net SENSOR_1: now also U4.GP26_A0; no longer U$1.GP26_A0
- net SENSOR_2: now also U4.GP27_A1; no longer U$1.GP27_A1
- net SENSOR_A: now also U4.GP12; no longer U$1.GP12
- net SENSOR_B: now also U4.GP13; no longer U$1.GP13
- net SENSOR_C: now also U4.GP14; no longer U$1.GP14
- net SS: now also U4.GP17; no longer U$1.GP17
- net T2: now also U4.GP0; no longer U$1.GP0
- net VCC: now also OUT_MOTOR_DRIVER.10, U4.VBUS, U5.VDD; no longer IC1.VDD, U$1.VBUS
- net V_COMP: now also U5.VOUT; no longer IC1.VOUT
Other:
- note added: "3V3 DCDC CONVERTER"
- note added: "3v3 para Filtro de ISENSE"
- note added: "CONTROL PANEL"
- note added: "DISPLAY OLED"
- note added: "HALL EFFECT SENSORS"
- note added: "HALL SIMULATOR"
- note added: "I2C BUS EXPANDER"
- note added: "IR SENSOR CONDITIONING"
- note added: "MOTOR DRIVER"
- note added: "MOTOR+HALL"
- note added: "RP PI PICO"
- note added: "SENSOR LENTO (medida en i2c expander)"
- note added: "SENSOR RAPIDO (medida en CPU)"
- note added: "TRIGGERS 1,2"
- moved on the sheet: C1, C10, C11, C12, C18, C2, C3, C4, C5, C6, C7, C8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

Commit message: Se pasa de 4 capas a 2 capas
El precio del prototipo es casi el doble con 4 caps
Changed lines of the file:
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@@
 <setting verticaltext="up"/>
 </settings>
-<grid distance="0.05" unitdist="inch" unit="inch" style="lines" multiple="1" display="no" altdistance="0.01" altunitdist="inch" altunit="inch"/>
+<grid distance="0.1" unitdist="inch" unit="inch" style="lines" multiple="1" display="no" altdistance="0.01" altunitdist="inch" altunit="inch"/>
 <layers>
 <layer number="1" name="Top" color="4" fill="1" visible="no" active="no"/>
@@
 <text x="270.51" y="-10.16" size="1.778" layer="97">SENSOR RAPIDO
 (medida en CPU)</text>
-<text x="-146.05" y="-11.43" size="1.778" layer="97">3v3 para Filtro de ISENSE</text>
+<text x="-143.51" y="-6.35" size="1.778" layer="97">3v3 para Filtro de ISENSE</text>
 </plain>
 <instances>

Commit message: ERC Pasado. Cambios menores
Al pasar el ERC se detecta fallo en la alimentacion del  pull-up de la linea de CS de la pantalla. Se soluciona cambiando a la alimentacion de 3v3.
Parts:
- renumbered IC2 to U6, IC3 to U7
Connections:
- removed net N$27: U7.P06
- removed net N$29: U7.P07
- removed net VCC-ISO: R66.1
- net VCC: now also R66.1
Other:
- moved on the sheet: R27
