File: 02.Hardware/PCBs/Tester Motor Faulhaber/TesterMotorFaulhaber.sch (EAGLE design)
At the start: 159 parts, among them J1 302-S201, J3 OSTVN03A150, Q1 2N7002PW, Q2 2N7002PW, Q3 2N7002PW, Q4 2N7002PW, Q5 2N7002PW, Q6 2N7002PW, Q7 2N7002PW, U1 MCP6071T-E/OT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

Commit message: PCB testeao de los motores faulhaber
Parts:
- R24, R26, R29, R33, R36, R38, R40: value (none) -> 100R
- R25, R28, R32, R34, R37, R39, R46: value (none) -> 10K
- R48, R52, R54: value 150 -> 150R
- R66: value 10k -> 10K
Other:
- note removed: "ISENSE = Iout * 0.025 * 25 = Iout *0.625"
- note removed: "OJO!! Es el de G=25 (TEUK version)"
