File: 02.Hardware/PCBs/Faulhaber Temp sensor  w CPU/Faulhaber Temp sensor  w CPU.sch (EAGLE design)
At the start: 16 parts, among them IC1 MCP9700T-E_TT, IC2 ATTINY85V-10SUR, Q2 SI2393DS-T1-GE3, Q3 2N7002PW, U7 AP2205-33W5-7

Commit message: Sensado de voltaje de entrada. version 2
Parts:
- added C8: 100n, SparkFun-Capacitors:0.1UF-0603-25V-(+80/-20%)
- added R3: (no value), SparkFun-Resistors:RESISTOR0603
- added R4: 169k, SparkFun-Resistors:RESISTOR0603
- added R5: 39k, SparkFun-Resistors:RESISTOR0603
- R1: value 100K -> (none)
- R2: value 33K -> (none)
Connections:
- new net N$1: IC1.VOUT, R3.1
- new net VOUTSENSE: C8.1, IC2.PB3_(PCINT3/XTAL1/CLKI/!OC1B!/ADC3), R4.2, R5.1
- net 3V3: now also R2.2
- net GND: now also C8.2, R5.2
- net ROJO: now also R4.1; no longer R2.2
- net SW_OUT: now also IC2.PB4_(PCINT4/XTAL2/CLKO/OC1B/ADC2); no longer IC2.PB1_(MISO/DO/AIN1/OC0B/OC1A/PCINT1)
- net USB+: now also IC2.PB1_(MISO/DO/AIN1/OC0B/OC1A/PCINT1); no longer IC2.PB3_(PCINT3/XTAL1/CLKI/!OC1B!/ADC3)
- net USB-: now also IC2.PB0_(MOSI/DI/SDA/AIN0/OC0A/!OC1A!/AREF/PCINT0); no longer IC2.PB4_(PCINT4/XTAL2/CLKO/OC1B/ADC2)
- net VTEMP: now also IC2.PB2_(SCK/USCK/SCL/ADC1/T0/INT0/PCINT2), R3.2; no longer IC1.VOUT, IC2.PB0_(MOSI/DI/SDA/AIN0/OC0A/!OC1A!/AREF/PCINT0)
Other:
- note added: "Faulhaber CPTemp v2_Abr'25"
- note added: "vo/vi = 0.1875 3.0 v @ vi=16v"
- note removed: "Faulhaber CPTemp v1_Mar'25"
- moved on the sheet: NEGRO, R2, ROJO
