File: 02.Hardware/Vanta Black/Vanta-Black v4/Vanta-Black v4.sch (EAGLE design)
At the start: 23 parts, among them U1 MCP9700T-E_TT, U2 AP2205-33W5-7, U3 MP6551GQB-Z, U4 ATTINY85V-10SUR

Commit message: VantaBlack v4
Parts:
- removed R1: 470k, SparkFun-Resistors:RESISTOR0603
- removed R2, R6: 10k, SparkFun-Resistors:RESISTOR0603
- added !RST, IN2: TESTPAD_TPSQB1,27, BeagleBone_Blue_R3:TESTPAD_TPSQB1,27
- added C8: 100n, SparkFun-Passives:CAP0805
- added R7: 5K6, SparkFun-Resistors:RESISTOR0603
- U3: value MP6551GQB-Z -> MP6614GN-Z; device SamacSys_Parts:MP6551GQB-Z -> SamacSys_Parts:MP6614GN-Z
- renumbered USB+ to VISEN, USB- to TX
Connections:
- removed net CM: R6.1, U3.CM1, U3.CM2
- removed net N$6: R1.1, U3.SR
- new net N$2: R7.2, U3.ISET
- net !RESET: now also !RST.TP
- net 3V3: no longer R2.2, U3.EN1, U3.EN2
- net GND: now also R7.1, U3.EP; no longer R1.2, R6.2
- net IN2: now also IN2.TP
- net MOT_OP+: now also C8.2, U3.OUT1; no longer U3.OUT1_1, U3.OUT1_2
- net MOT_OP-: now also C8.1, U3.OUT2; no longer U3.OUT2_1, U3.OUT2_2
- net NFAULT: now also U3.VISEN; no longer R2.1, U3.NFAULT, VISEN.TP
- net VTEMP: now also VISEN.TP
Other:
- note added: "VANTA BLACK v4_oct25"
- note removed: "CM (current measurement) Tarado a 3.3 A"
- note removed: "Low --> *Overcurrent *Overtemperature"
- note removed: "SR (Slew Rate) 470k --> 1.5 us"
- note removed: "VANTA BLACK v2_Jun'25"
