File: 02.Hardware/PCBs/Faulhaber w CPU switchoutput/Faulhaber w CPU switchoutput.brd (EAGLE design)
At the start: 21.9 x 23.6 mm, 22 parts, among them U1 MCP9700T-E_TT, U2 AP2205-33W5-7, U3 MP6551GQB-Z, U4 ATTINY85V-10SUR

Commit message: PCBs
Parts:
- added C3: 2.2u, SparkFun-Capacitors:0603-CAP
- C4: value 100n 50v -> 2.2u; device adafruit:C0805 -> SparkFun-Capacitors:0603-CAP
- C5: value 1u -> 100n
- R1: value 0R -> 470k
- R2, R6: value 0R -> 10k
- R3: value (none) -> 2k2
- moved C1 5.35 mm to (115.6, 89.3)
- moved C5 4.63 mm to (110.6, 89.4)
- moved C2 0.66 mm to (113.2, 89.2)
- moved R6 0.64 mm to (105.1, 79.0)
- moved C4 0.16 mm to (100.2, 90.0)
Connections:
- net GND_OUT renamed MOT_OP-
- removed net VCC: U3.10
- removed net VMOT+: U3.1
- new net !RESET: U4.1
- new net MOT_OP+: U3.1, U3.10
- net 3V3: now also C3.1
- net GND: now also C3.2; no longer U2.3
- net VROVER+: now also U2.3
Routing:
- net VROVER+: track 44.4 -> 59.9 mm
- net MOT_OP+: track 0.00 -> 10.5 mm, vias 0 -> 3
- net VCC: track 7.71 -> 0.00 mm, vias 3 -> 0
- net MOT_OP-: track 0.00 -> 4.63 mm
- net GND: track 55.2 -> 53.7 mm
- net 3V3: track 54.9 -> 56.4 mm
- net CM: track 13.4 -> 14.2 mm, vias 2 -> 3
- added copper zone on layer 1, net MOT_OP+
- added copper zone on layer 16, net MOT_OP+
- removed copper zone on layer 1, net VCC
- removed copper zone on layer 16, net VCC
Other:
- board text added: "Faulhaber CPU SWITCH v2_Jun'25"
- board text removed: "Faulhaber CPU SWITCH v1_Abr'25"
