File: 02.Hardware/PCBs/Faulhaber w CPU switchoutput/Faulhaber w CPU switchoutput.sch (EAGLE design)
At the start: 22 parts, among them U1 MCP9700T-E_TT, U2 AP2205-33W5-7, U3 MP6551GQB-Z, U4 ATTINY85V-10SUR

Commit message: PCBs
Parts:
- added C3: 2.2u, SparkFun-Capacitors:4.7UF-6.3V-10%(0603)0603
- C4: value 100n 50v -> 2.2u; device adafruit:C-USC0805 -> SparkFun-Capacitors:4.7UF-6.3V-10%(0603)0603
- C5: value 1u -> 100n
- R1: value 0R -> 470k
- R2, R6: value 0R -> 10k
- R3: value (none) -> 2k2
Connections:
- net GND_OUT renamed MOT_OP-
- removed net VCC: U3.OUT1_2
- removed net VMOT+: U3.OUT1_1
- new net !RESET: U4.PB5_(PCINT5/!RESET!/ADC0/DW)
- new net MOT_OP+: U3.OUT1_1, U3.OUT1_2
- net 3V3: now also C3.1
- net GND: now also C3.2; no longer U2.EN
- net VROVER+: now also U2.EN
Other:
- note added: "CM (current measurement) Tarado a 3.3 A"
- note added: "Faulhaber CPU SWITCH v2_Jun'25"
- note added: "Low --> *Overcurrent *Overtemperature"
- note added: "R para aislar SCK_SPI de programacion de la salida del sensor de temperatura"
- note added: "SR (Slew Rate) 470k --> 1.5 us"
- note added: "Test Pads"
- note added: "Vout sense Tarado @ Vsense=14.3v --> Vin=3.3v"
- note removed: "3V (pq no tenian 3.3V en stock)"
- note removed: "Faulhaber CPU SWITCH v1_Abr'25"
- moved on the sheet: C4, C5, R1, R2, R6, U3, VROVER+
