File: 02.Hardware/PCBs/TestMachines/Test Machines.brd (EAGLE design)
At the start: 122 x 120 mm, 175 parts, among them IC1 MCP23017SO, IC2 ULN2803CDWR, IC3 ULN2803CDWR, K1 J1031C3VDC.15S, K10 J1031C3VDC.15S, K11 J1031C3VDC.15S, K12 J1031C3VDC.15S, K13 J1031C3VDC.15S, K14 J1031C3VDC.15S, K15 J1031C3VDC.15S, K16 J1031C3VDC.15S, K17 J1031C3VDC.15S, K18 J1031C3VDC.15S, K2 J1031C3VDC.15S, K3 J1031C3VDC.15S, K4 J1031C3VDC.15S, K5 J1031C3VDC.15S, K6 J1031C3VDC.15S, K7 J1031C3VDC.15S, K8 J1031C3VDC.15S, K9 J1031C3VDC.15S, Q1 2N7002PW, Q2 2N7002PW, Q3 2N7002PW, Q4 2N7002PW, Q5 2N7002PW, Q6 2N7002PW, U12 AP64501SP-13, U15 NTMS4801NR2G, U17 AP63203, U2 MCP4725, U5 MCP6071T-E/OT, U6 MCP6071T-E/OT, U7 TPIC2810D

Commit message: Versiones enviadas a PCB way
Parts:
- added D22, D23: STPS1L40U, STPS1L40U:SMB_STM
- moved R66 2.77 mm to (99.8, 35.1)
- moved R61 2.70 mm to (99.2, 32.6)
Connections:
- net N$14: now also D22.1
- net N$15: now also D23.1
- net VCC: now also D22.2, D23.2
Routing:
- net VBUS: track 384.4 -> 377.5 mm
- net VCC: track 102.0 -> 108.9 mm
- net SS: track 45.8 -> 39.3 mm
- net V_MOT_SENSE: track 465.0 -> 469.6 mm
- net N$15: track 25.2 -> 29.0 mm
- net N$14: track 7.75 -> 11.0 mm
- net EN_DCDC: track 111.7 -> 109.2 mm
- net SDA: track 172.9 -> 171.2 mm
- net N$90: track 26.1 -> 27.4 mm
- net SCL: track 149.5 -> 148.3 mm
- net SCK: track 23.7 -> 22.7 mm
- net IMOTOR: track 144.5 -> 143.5 mm
- net N$91: track 24.6 -> 25.5 mm
- net N$92: track 23.1 -> 23.8 mm
- net N$105: track 25.4 -> 26.0 mm
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Other:
- board text added: "TestMachine v1-Mar'25"
- board text removed: "TestMachine v1-Feb'25"

Commit message: PCBs
Parts:
- R10: value (none) -> 22k
- R11: value (none) -> 15k
- R18: value (none) -> 5k1
- R19: value (none) -> 8k2
- R20: value (none) -> 2k4
- R21: value (none) -> 62k
- R22: value (none) -> 4k3
- R23: value (none) -> 36k
- R27: value (none) -> 1k
- R3, R43: value (none) -> 11k
- R30, R45: value (none) -> N.C
- R4: value (none) -> 5k6
- R41: value (none) -> 150k
- R42, R66: value (none) -> 10k
- R44: value (none) -> 25k
- R5: value (none) -> 2k8
- R55, R56, R57, R59, R61: value (none) -> 33
- R6: value (none) -> 1k4
- R7: value (none) -> 180k
- R8: value (none) -> 91k
- R9: value (none) -> 43k
- RSENSE1: value (none) -> 100mR
